Commit message: added readme, correctly rotated cylinder

File: urdf/amarsmer.xacro (robot description, xacro)
@@ -27,5 +27,5 @@
     <inertial>
         <mass value="${mass}"/>
-        <origin xyz="0 0 ${z_cog}"/>
+        <origin xyz="0 0 ${z_cog}" rpy="0 ${pi/2} 0"/>
     <!-- BlueROV2 values from "Model Predictive Control for the BlueROV2",
         Emil Már Einarsson, Andris Lipenitis, Master thesis, 2020
@@ -40,4 +40,5 @@
     </inertial>
     <visual>
+    <origin rpy="0 ${pi/2} 0" xyz="0 0 0"/>
       <geometry>
         <cylinder length="0.6" radius="0.2"/>
@@ -60,5 +61,5 @@
     </link>
 <xacro:include filename="hydrodynamics.xacro"/>
-<xacro:include filename="thrusters.xacro"/>
+<xacro:include filename="thrusters_plasmar2.xacro"/>
 <!-- other Gazebo plugins -->
 <xacro:if value="$(arg simulation)">
