Commit message: Removed mechanical limits (set arbitrarily high) on steering joints.

File: amarsmer_description/urdf/thrusters_plasmar2.xacro (robot description, xacro)
@@ -49,5 +49,5 @@
       <parent link="${ns}/base_link" />
       <child link="${ns}/thruster${thruster_id}_steering" />
-      <limit effort="100" velocity="40" lower="${-pi/2}" upper="${pi/2}"/>
+      <limit effort="100" velocity="40" lower="-1e16" upper="1e16"/>
     </joint>
     <!-- Joint between thruster link and vehicle base link -->
