Commit message: cloned the updated repo and manually added the previously changed files (quick and dirty but manageable for now)

File: amarsmer_description/urdf/amarsmer.xacro (robot description, xacro)
@@ -61,5 +61,5 @@
     </link>
 <xacro:include filename="hydrodynamics.xacro"/>
-<xacro:include filename="thrusters_plasmar2.xacro"/>
+<xacro:include filename="thrusters_plasmar1a.xacro"/>
 <!-- other Gazebo plugins -->
 <xacro:if value="$(arg simulation)">

File: amarsmer_description/urdf/thrusters_plasmar1a.xacro (robot description, xacro)
@@ -66,8 +66,8 @@
   </xacro:thruster>
   <xacro:thruster thruster_id="3">
-    <origin xyz="${cylinder_l/4} 0 -${cylinder_r}" rpy="0 0 ${pi/2}"/>
+    <origin xyz="${cylinder_l/4} -${cylinder_r} 0" rpy="0 ${pi/2} 0"/>
   </xacro:thruster>
   <xacro:thruster thruster_id="4">
-    <origin xyz="${cylinder_l/4} 0 ${cylinder_r}" rpy="0 0 ${pi/2}"/>
+    <origin xyz="${cylinder_l/4} ${cylinder_r} 0" rpy="0 ${pi/2} 0"/>
   </xacro:thruster>
 </robot>

File: amarsmer_description/urdf/thrusters_plasmar2.xacro (robot description, xacro)
@@ -6,5 +6,5 @@
   <xacro:property name="prop_l" value="0.035"/>
   <xacro:property name="cylinder_l" value="0.6"/>
-   <xacro:property name="cylinder_r" value="0.2"/>
+   <xacro:property name="cylinder_r" value="0.25"/>
   <!--  Thruster macro: joint + link + plugin -->
   <xacro:macro name="thruster" params="thruster_id *origin">
@@ -91,5 +91,5 @@
 </gazebo>
 </xacro:macro>
-  <!-- all 6 thrusters -->
+  <!-- all 4 thrusters -->
   <xacro:thruster thruster_id="1">
     <origin xyz="-${cylinder_l/2} -${cylinder_r} 0" rpy="0 0 -${pi/2}"/>

Commit message: added wrench display

File: amarsmer_description/urdf/amarsmer.xacro (robot description, xacro)
@@ -43,5 +43,5 @@
     <origin rpy="0 ${pi/2} 0" xyz="0 0 0"/>
       <geometry>
-        <cylinder length="0.6" radius="0.2"/>
+        <cylinder length="0.6" radius="0.1"/>
       </geometry>
       <material name="color"/>

File: amarsmer_description/urdf/thrusters_plasmar2.xacro (robot description, xacro)
@@ -6,5 +6,5 @@
   <xacro:property name="prop_l" value="0.035"/>
   <xacro:property name="cylinder_l" value="0.6"/>
-   <xacro:property name="cylinder_r" value="0.25"/>
+   <xacro:property name="cylinder_r" value="0.15"/>
   <!--  Thruster macro: joint + link + plugin -->
   <xacro:macro name="thruster" params="thruster_id *origin">
@@ -41,5 +41,5 @@
       <inertia  izz="0.1" ixy="0.0"  ixz="0.0"
                 iyy="0.1" iyz="0.0"
-                ixx="0.1" />
+                ixx="0.1" />ros2gz
     </inertial>
     </link>
@@ -99,8 +99,8 @@
   </xacro:thruster>
   <xacro:thruster thruster_id="3">
-    <origin xyz="${cylinder_l/2} 0 -${cylinder_r}" rpy="${pi/2} ${pi/2} 0"/>
+    <origin xyz="0 0 -${cylinder_r}" rpy="${pi/2} ${pi/2} 0"/>
   </xacro:thruster>
   <xacro:thruster thruster_id="4">
-    <origin xyz="${cylinder_l/2} 0 ${cylinder_r}" rpy="-${pi/2} -${pi/2} 0"/>
+    <origin xyz="0 0 ${cylinder_r}" rpy="-${pi/2} -${pi/2} 0"/>
   </xacro:thruster>
 </robot>

Commit message: edited robot model, added node that converts pose in quaternion to rpy

File: amarsmer_description/urdf/amarsmer.xacro (robot description, xacro)
@@ -19,5 +19,5 @@
   <xacro:property name="prop_mass" value="0.07"/>
   <!-- to set correct buoyancy volume with 1 % positive factor -->
-  <xacro:property name="buoyant_correction" value="${1.01*pow((mass + 6*prop_mass)/(density*x_size*y_size*z_size), 1./3)}"/>
+  <xacro:property name="buoyant_correction" value="${1.01*pow((mass + 4*prop_mass)/(density*x_size*y_size*z_size), 1./3)}"/>
   <!-- Center of buoyancy -->
   <xacro:property name="z_cob" value="${-buoyant_correction*z_size/4}"/>

File: amarsmer_description/urdf/thrusters_plasmar2.xacro (robot description, xacro)
@@ -49,5 +49,5 @@
       <parent link="${ns}/base_link" />
       <child link="${ns}/thruster${thruster_id}_steering" />
-      <limit effort="100" velocity="40" lower="${-pi/4}" upper="${pi/4}"/>
+      <limit effort="100" velocity="40" lower="${-pi/2}" upper="${pi/2}"/>
     </joint>
     <!-- Joint between thruster link and vehicle base link -->
@@ -78,6 +78,6 @@
             <velocity_control>true</velocity_control>
             <use_angvel_cmd>false</use_angvel_cmd>
-            <max_thrust_cmd>40</max_thrust_cmd>
-            <min_thrust_cmd>-40</min_thrust_cmd>
+            <max_thrust_cmd>400</max_thrust_cmd>
+            <min_thrust_cmd>-400</min_thrust_cmd>
         </plugin>
     <plugin filename="ignition-gazebo-joint-position-controller-system" name="ignition::gazebo::systems::JointPositionController">
@@ -99,8 +99,8 @@
   </xacro:thruster>
   <xacro:thruster thruster_id="3">
-    <origin xyz="0 0 -${cylinder_r}" rpy="${pi/2} ${pi/2} 0"/>
+    <origin xyz="0 0 -${cylinder_r}" rpy="${pi/2} ${pi/2} ${pi/2}"/>
   </xacro:thruster>
   <xacro:thruster thruster_id="4">
-    <origin xyz="0 0 ${cylinder_r}" rpy="-${pi/2} -${pi/2} 0"/>
+    <origin xyz="0 0 ${cylinder_r}" rpy="-${pi/2} -${pi/2} ${pi/2}"/>
   </xacro:thruster>
 </robot>

Commit message: Major overhaul of code architecture to make it easier to use and to add new features

File: amarsmer_description/urdf/amarsmer.xacro (robot description, xacro)
@@ -15,6 +15,16 @@
   <xacro:property name="y_size" value="0.25"/>
   <xacro:property name="z_size" value="0.1"/>
-  <xacro:property name="mass" value="14.8"/>
+  <!-- Read main yaml file for inertia and mass -->
+  <xacro:arg name="config_file"
+             default="$(find amarsmer_control)/config/robot.yaml"/>
+  <xacro:property name="config_path"
+                  value="$(arg config_file)"/>
+  <xacro:property name="cfg"
+                  value="${xacro.load_yaml(config_path)}"/>
+  <xacro:property name="robot"
+                  value="${cfg['robot']}"/>
   <!-- other props -->
+  <xacro:property name="mass"
+                value="${robot['mass']}"/>
   <xacro:property name="prop_mass" value="0.07"/>
   <!-- to set correct buoyancy volume with 1 % positive factor -->
@@ -24,19 +34,17 @@
   <!-- Center of gravity -->
   <xacro:property name="z_cog" value="${-buoyant_correction*z_size}"/>
+  <!-- <link name="${ns}/base_link"> -->
   <!-- Vehicle base link -->
     <link name="${ns}/base_link">
     <inertial>
-        <mass value="${mass}"/>
+        <mass value="${robot['mass']}"/>
         <origin xyz="0 0 ${z_cog}" rpy="0 ${pi/2} 0"/>
-    <!-- BlueROV2 values from "Model Predictive Control for the BlueROV2",
-        Emil Már Einarsson, Andris Lipenitis, Master thesis, 2020
-        for now make Ignition crash?-->
-<!--         <inertia ixx="0.21" ixy="0.00" ixz="0.00" iyy="0.245" iyz="0.00" izz="0.245"/> -->
-        <inertia ixx="5.2539" ixy="0.0144" ixz="0.3341" iyy="7.9420" iyz="0.026" izz="6.9123"/>
-            <!-- Perfect rectangle -->
-<!--        <inertia
-        ixx="${mass/12*(y_size*y_size+z_size*z_size)}" ixy="0.0" ixz="0.0"
-        iyy="${mass/12*(x_size*x_size + z_size*z_size)}" iyz="0.0"
-        izz="${mass/12*(x_size*x_size + y_size*y_size)}" />-->
+        <inertia
+        ixx="${robot['inertia']['ixx']}"
+        ixy="${robot['inertia']['ixy']}"
+        ixz="${robot['inertia']['ixz']}"
+        iyy="${robot['inertia']['iyy']}"
+        iyz="${robot['inertia']['iyz']}"
+        izz="${robot['inertia']['izz']}"/>
     </inertial>
     <visual>

File: amarsmer_description/urdf/hydrodynamics.xacro (robot description, xacro)
@@ -1,51 +1,35 @@
 <?xml version="1.0"?>
-<xacro>
-<gazebo>
-    <plugin filename="ignition-gazebo-hydrodynamics-system" name="ignition::gazebo::systems::Hydrodynamics">
-<!--     <density>${density}</density> -->
-    <!-- Ignition notations from Handbook of Marine Craft, Fossen, 2011 -->
-    <link_name>${ns}/base_link</link_name>
-    <!-- BlueROV2 heavy values from "6-DoF Modelling and Control of a Remotely Operated Vehicle"
-        Wu, Master thesis, Flinder University, 2018  -->
-    <!-- Negative diagonal values of added mass matrix [Fossen (6.38)] -->
-    <xDotU>-5.5</xDotU>
-    <yDotV>-12.7</yDotV>
-    <zDotW>-14.57</zDotW>
-    <kDotP>-0.12</kDotP>
-    <mDotQ>-0.12</mDotQ>
-    <nDotR>-0.12</nDotR>
-    <!-- From "Numerical Modelling and Experimental Testing of the Hydrodynamic Characteristics
-        for an Open-Frame Remotely Operated Vehicle",  Li et al, Marine Science and Engineering, 2020         -->
-    <!-- Negative linear damping [Fossen (6.62)] -->
-<!--    <xU>-1.31</xU>
-    <yV>-9.14</yV>
-    <zW>-2.015</zW>
-    <kP>-0.</kP>
-    <mQ>-0.</mQ>
-    <nR>-0.</nR>-->
-    <!-- Negative quadratic damping [Fossen (6.62)] -->
-      <xUabsU>-33.800000000000004</xUabsU>
-      <yVabsV>-54.26875</yVabsV>
-      <zWabsW>-73.37135</zWabsW>
-      <kPabsP>-40.0</kPabsP>
-      <mQabsQ>-40.0</mQabsQ>
-      <nRabsR>-40.0</nRabsR>
-    <!-- BlueROV2 values from "Model Predictive Control for the BlueROV2",
-        Emil Már Einarsson, Andris Lipenitis, Master thesis, 2020  -->
-    <!-- Negative linear damping -->
-    <xU>-25.15</xU>
-    <yV>-7.364</yV>
-    <zW>-17.955</zW>
-    <kP>-10.888</kP>
-    <mQ>-20.761</mQ>
-    <nR>-3.744</nR>
-    <!-- Negative quadratic damping -->
-<!--    <xUU>-17.77</xUU>
-    <yVV>-125.9</yVV>
-    <zWW>-72.36</zWW>
-    <kPP>-0.1246</kPP>
-    <mQQ>-0.1246</mQQ>
-    <nRR>-0.1857</nRR>-->
+<xacro xmlns:xacro="http://www.ros.org/wiki/xacro">
+  <!-- Load YAML -->
+  <xacro:property name="cfg"
+                value="${xacro.load_yaml('$(find amarsmer_control)/config/robot.yaml')}"/>
+<xacro:property name="hydro"
+                value="${cfg['hydrodynamics']}"/>
+  <gazebo>
+    <plugin filename="ignition-gazebo-hydrodynamics-system"
+            name="ignition::gazebo::systems::Hydrodynamics">
+      <link_name>${ns}/base_link</link_name>
+      <!-- Added mass -->
+      <xDotU>${hydro['added_mass']['xDotU']}</xDotU>
+      <yDotV>${hydro['added_mass']['yDotV']}</yDotV>
+      <zDotW>${hydro['added_mass']['zDotW']}</zDotW>
+      <kDotP>${hydro['added_mass']['kDotP']}</kDotP>
+      <mDotQ>${hydro['added_mass']['mDotQ']}</mDotQ>
+      <nDotR>${hydro['added_mass']['nDotR']}</nDotR>
+      <!-- Quadratic damping -->
+      <xUabsU>${hydro['quadratic_damping']['xUabsU']}</xUabsU>
+      <yVabsV>${hydro['quadratic_damping']['yVabsV']}</yVabsV>
+      <zWabsW>${hydro['quadratic_damping']['zWabsW']}</zWabsW>
+      <kPabsP>${hydro['quadratic_damping']['kPabsP']}</kPabsP>
+      <mQabsQ>${hydro['quadratic_damping']['mQabsQ']}</mQabsQ>
+      <nRabsR>${hydro['quadratic_damping']['nRabsR']}</nRabsR>
+      <!-- Linear damping -->
+      <xU>${hydro['linear_damping']['xU']}</xU>
+      <yV>${hydro['linear_damping']['yV']}</yV>
+      <zW>${hydro['linear_damping']['zW']}</zW>
+      <kP>${hydro['linear_damping']['kP']}</kP>
+      <mQ>${hydro['linear_damping']['mQ']}</mQ>
+      <nR>${hydro['linear_damping']['nR']}</nR>
     </plugin>
-</gazebo>
+  </gazebo>
 </xacro>

File: amarsmer_description/urdf/thrusters_plasmar_ur.xacro (robot description, xacro)
@@ -5,13 +5,16 @@
   <xacro:property name="prop_r" value="0.05"/>
   <xacro:property name="prop_l" value="0.035"/>
+  <xacro:property name="cylinder_l" value="0.6"/>
+   <xacro:property name="cylinder_r" value="0.15"/>
   <!--  Thruster macro: joint + link + plugin -->
   <xacro:macro name="thruster" params="thruster_id *origin">
     <link name="${ns}/thruster${thruster_id}">
       <visual>
+        <origin xyz="0 0 0" rpy="1.5708 0 0"/>  <!-- Rotate thruster 90° around X -->
         <geometry>
-          <xacro:if value="${thruster_id in [1,2,5]}">
+          <xacro:if value="${thruster_id in [1,2]}">
             <mesh filename="${prop_mesh_cw}"/>
           </xacro:if>
-            <xacro:unless value="${thruster_id in [1,2,5]}">
+          <xacro:unless value="${thruster_id in [1,2]}">
             <mesh filename="${prop_mesh_ccw}"/>
           </xacro:unless>
@@ -25,6 +28,5 @@
       </collision>-->
      <inertial>
-     <!-- thruster axis is X -->
-      <origin xyz="${prop_l/2} 0 0" rpy="0 0 0" />
+      <origin xyz="${prop_l/2} 0 0" rpy="1.5708 0 0" />  <!-- Rotate inertia 90° around X -->
       <mass value="${prop_mass}" />
       <inertia  izz="${prop_mass*prop_r*prop_r / 4  + prop_mass*prop_l*prop_l / 12}" ixy="0.0"  ixz="0.0"
@@ -39,21 +41,21 @@
       <inertia  izz="0.1" ixy="0.0"  ixz="0.0"
                 iyy="0.1" iyz="0.0"
-                ixx="0.1" />
+                ixx="0.1" />ros2gz
     </inertial>
     </link>
     <joint name="thruster${thruster_id}_steering" type="revolute">
       <xacro:insert_block name="origin" />
-        <axis xyz="1 0 0" />
+        <axis xyz="1 0 0" rpy="0 0 0"/>
       <parent link="${ns}/base_link" />
       <child link="${ns}/thruster${thruster_id}_steering" />
-      <limit effort="100" velocity="40" lower="${-pi/4}" upper="${pi/4}"/>
+      <limit effort="100" velocity="40" lower="-1e16" upper="1e16"/>
     </joint>
     <!-- Joint between thruster link and vehicle base link -->
     <joint name="thruster${thruster_id}" type="continuous">
-<!--       <xacro:insert_block name="origin" /> -->
+      <origin xyz="0 0 0" rpy="0 0 1.5708"/>  <!-- 90° offset along Z -->
       <xacro:if value="${thruster_id in [1,2,5]}">
         <axis xyz="1 0 0" />
       </xacro:if>
-      <xacro:unless value="${thruster_id in [1,2,5]}">
+      <xacro:unless value="${thruster_id in [3,4,6]}">
         <axis xyz="-1 0 0" />
       </xacro:unless>
@@ -76,6 +78,6 @@
             <velocity_control>true</velocity_control>
             <use_angvel_cmd>false</use_angvel_cmd>
-            <max_thrust_cmd>40</max_thrust_cmd>
-            <min_thrust_cmd>-40</min_thrust_cmd>
+            <max_thrust_cmd>400</max_thrust_cmd>
+            <min_thrust_cmd>-400</min_thrust_cmd>
         </plugin>
     <plugin filename="ignition-gazebo-joint-position-controller-system" name="ignition::gazebo::systems::JointPositionController">
@@ -89,22 +91,10 @@
 </gazebo>
 </xacro:macro>
-  <!-- all 6 thrusters -->
+  <!-- all thrusters -->
   <xacro:thruster thruster_id="1">
-    <origin xyz="0.1355 -0.1 -0.0725" rpy="0 0 0.7853981634"/>
+    <origin xyz="-${cylinder_l/2} -${cylinder_r} 0" rpy="0 0 -${pi/2}"/>
   </xacro:thruster>
   <xacro:thruster thruster_id="2">
-    <origin xyz="0.1355 0.1 -0.0725" rpy="0 0 -0.7853981634"/>
-  </xacro:thruster>
-  <xacro:thruster thruster_id="3">
-    <origin xyz="-0.1475 -0.1 -0.0725" rpy="0 0 2.3561944902"/>
-  </xacro:thruster>
-  <xacro:thruster thruster_id="4">
-    <origin xyz="-0.1475 0.1 -0.0725" rpy="0 0 -2.3561944902"/>
-  </xacro:thruster>
-  <xacro:thruster thruster_id="5">
-    <origin xyz="0.0025 -0.1105 -0.005" rpy="0 -1.5707963268 0"/>
-  </xacro:thruster>
-  <xacro:thruster thruster_id="6">
-    <origin xyz="0.0025 0.1105 -0.005" rpy="0 -1.5707963268 0"/>
+    <origin xyz="-${cylinder_l/2} ${cylinder_r} 0" rpy="${pi} 0 ${pi/2}"/>
   </xacro:thruster>
 </robot>

File: amarsmer_description/urdf/thrusters_plasmar_uvr.xacro (robot description, xacro)
@@ -91,5 +91,5 @@
 </gazebo>
 </xacro:macro>
-  <!-- all 4 thrusters -->
+  <!-- all thrusters -->
   <xacro:thruster thruster_id="1">
     <origin xyz="-${cylinder_l/2} -${cylinder_r} 0" rpy="0 0 -${pi/2}"/>
