Commit message: Added blueROV2 architecture back (not implemented in control yet)

File: amarsmer_description/urdf/thrusters_blueROV2.xacro (robot description, xacro)
@@ -1,20 +1,17 @@
 <?xml version="1.0"?>
 <robot xmlns:xacro="http://www.ros.org/wiki/xacro">
-  <xacro:property name="prop_mesh_cw" value="package://amarsmer_description/meshes/bluerov2_propcw.dae"/>
-  <xacro:property name="prop_mesh_ccw" value="package://amarsmer_description/meshes/bluerov2_propccw.dae"/>
+  <xacro:property name="prop_mesh_cw" value="package://bluerov2_description/meshes/bluerov2_propcw.dae"/>
+  <xacro:property name="prop_mesh_ccw" value="package://bluerov2_description/meshes/bluerov2_propccw.dae"/>
   <xacro:property name="prop_r" value="0.05"/>
   <xacro:property name="prop_l" value="0.035"/>
-  <xacro:property name="cylinder_l" value="0.6"/>
-   <xacro:property name="cylinder_r" value="0.15"/>
   <!--  Thruster macro: joint + link + plugin -->
   <xacro:macro name="thruster" params="thruster_id *origin">
     <link name="${ns}/thruster${thruster_id}">
       <visual>
-        <origin xyz="0 0 0" rpy="1.5708 0 0"/>  <!-- Rotate thruster 90° around X -->
         <geometry>
           <xacro:if value="${thruster_id in [1,2,5]}">
             <mesh filename="${prop_mesh_cw}"/>
           </xacro:if>
-          <xacro:unless value="${thruster_id in [1,2,5]}">
+            <xacro:unless value="${thruster_id in [1,2,5]}">
             <mesh filename="${prop_mesh_ccw}"/>
           </xacro:unless>
@@ -28,5 +25,6 @@
       </collision>-->
      <inertial>
-      <origin xyz="${prop_l/2} 0 0" rpy="1.5708 0 0" />  <!-- Rotate inertia 90° around X -->
+     <!-- thruster axis is X -->
+      <origin xyz="${prop_l/2} 0 0" rpy="0 0 0" />
       <mass value="${prop_mass}" />
       <inertia  izz="${prop_mass*prop_r*prop_r / 4  + prop_mass*prop_l*prop_l / 12}" ixy="0.0"  ixz="0.0"
@@ -35,32 +33,16 @@
     </inertial>
     </link>
-      <!-- Joint between thruster attach point and vehicle base link -->
-    <link name="${ns}/thruster${thruster_id}_steering">
-      <inertial>
-      <mass value="0.1" />
-      <inertia  izz="0.1" ixy="0.0"  ixz="0.0"
-                iyy="0.1" iyz="0.0"
-                ixx="0.1" />ros2gz
-    </inertial>
-    </link>
-    <joint name="thruster${thruster_id}_steering" type="revolute">
-      <xacro:insert_block name="origin" />
-        <axis xyz="1 0 0" rpy="0 0 0"/>
-      <parent link="${ns}/base_link" />
-      <child link="${ns}/thruster${thruster_id}_steering" />
-      <limit effort="100" velocity="40" lower="-1e16" upper="1e16"/>
-    </joint>
     <!-- Joint between thruster link and vehicle base link -->
     <joint name="thruster${thruster_id}" type="continuous">
-      <origin xyz="0 0 0" rpy="0 0 1.5708"/>  <!-- 90° offset along Z -->
+      <xacro:insert_block name="origin" />
       <xacro:if value="${thruster_id in [1,2,5]}">
         <axis xyz="1 0 0" />
       </xacro:if>
-      <xacro:unless value="${thruster_id in [3,4,6]}">
+      <xacro:unless value="${thruster_id in [1,2,5]}">
         <axis xyz="-1 0 0" />
       </xacro:unless>
-      <parent link="${ns}/thruster${thruster_id}_steering" />
+      <parent link="${ns}/base_link" />
       <child link="${ns}/thruster${thruster_id}" />
-      <limit effort="-1" velocity="-1"/>
+      <limits effort="-1" velocity="-1"/>
     </joint>
     <!-- ignition topic is /model/{ns}/joint/{joint_name}/cmd_pos -->
@@ -78,29 +60,28 @@
             <velocity_control>true</velocity_control>
             <use_angvel_cmd>false</use_angvel_cmd>
-            <max_thrust_cmd>400</max_thrust_cmd>
-            <min_thrust_cmd>-400</min_thrust_cmd>
+            <max_thrust_cmd>40</max_thrust_cmd>
+            <min_thrust_cmd>-40</min_thrust_cmd>
         </plugin>
-    <plugin filename="ignition-gazebo-joint-position-controller-system" name="ignition::gazebo::systems::JointPositionController">
-        <joint_name>thruster${thruster_id}_steering</joint_name>
-        <p_gain>10.</p_gain>
-        <i_gain>0.2</i_gain>
-        <d_gain>0.1</d_gain>
-        <i_max>10</i_max>
-        <i_min>-10</i_min>
-      </plugin>
-</gazebo>
+      </gazebo>
+<!--  </xacro:if> -->
 </xacro:macro>
-  <!-- all 4 thrusters -->
+  <!-- all 6 thrusters -->
   <xacro:thruster thruster_id="1">
-    <origin xyz="-${cylinder_l/2} -${cylinder_r} 0" rpy="0 0 -${pi/2}"/>
+    <origin xyz="0.1355 -0.1 -0.0725" rpy="0 0 0.7853981634"/>
   </xacro:thruster>
   <xacro:thruster thruster_id="2">
-    <origin xyz="-${cylinder_l/2} ${cylinder_r} 0" rpy="${pi} 0 ${pi/2}"/>
+    <origin xyz="0.1355 0.1 -0.0725" rpy="0 0 -0.7853981634"/>
   </xacro:thruster>
   <xacro:thruster thruster_id="3">
-    <origin xyz="0 0 -${cylinder_r}" rpy="${pi/2} ${pi/2} ${pi/2}"/>
+    <origin xyz="-0.1475 -0.1 -0.0725" rpy="0 0 2.3561944902"/>
   </xacro:thruster>
   <xacro:thruster thruster_id="4">
-    <origin xyz="0 0 ${cylinder_r}" rpy="-${pi/2} -${pi/2} ${pi/2}"/>
+    <origin xyz="-0.1475 0.1 -0.0725" rpy="0 0 -2.3561944902"/>
+  </xacro:thruster>
+  <xacro:thruster thruster_id="5">
+    <origin xyz="0.0025 -0.1105 -0.005" rpy="0 -1.5707963268 0"/>
+  </xacro:thruster>
+  <xacro:thruster thruster_id="6">
+    <origin xyz="0.0025 0.1105 -0.005" rpy="0 -1.5707963268 0"/>
   </xacro:thruster>
 </robot>
